Commit message: Sync runtime with ver6 robot hardware

File: urdf/biped_bike_runtime.urdf (robot description, URDF)
Before this commit: robot biped_bike_robot_ver5, 21 links, 20 joints
Links:
- link arm_base_yaw: geometry collision mesh filename=package://biped_bike_runtime/meshes/arm_base_yaw.STL; visual mesh filename=package://biped_bike_runtime/meshes/arm_base_yaw.STL
- link arm_elbow_pitch: geometry collision mesh filename=package://biped_bike_runtime/meshes/arm_elbow_pitch.STL; visual mesh filename=package://biped_bike_runtime/meshes/arm_elbow_pitch.STL
- link arm_shoulder_pitch: mass 0.10092 -> 0.10542; geometry collision mesh filename=package://biped_bike_runtime/meshes/arm_shoulder_pitch.STL; visual mesh filename=package://biped_bike_runtime/meshes/arm_shoulder_pitch.STL
- link arm_wrist_pitch: geometry collision mesh filename=package://biped_bike_runtime/meshes/arm_wrist_pitch.STL; visual mesh filename=package://biped_bike_runtime/meshes/arm_wrist_pitch.STL
- link arm_wrist_roll: geometry collision mesh filename=package://biped_bike_runtime/meshes/arm_wrist_roll.STL; visual mesh filename=package://biped_bike_runtime/meshes/arm_wrist_roll.STL
- link base_link: mass 0.63285 -> 0.62617; geometry collision mesh filename=package://biped_bike_runtime/meshes/base_link.STL; visual mesh filename=package://biped_bike_runtime/meshes/base_link.STL
- link l_ankle_pitch: geometry collision mesh filename=package://biped_bike_runtime/meshes/l_ankle_pitch.STL; visual mesh filename=package://biped_bike_runtime/meshes/l_ankle_pitch.STL
- link l_foot_roll: geometry collision mesh filename=package://biped_bike_runtime/meshes/l_foot_roll.STL; visual mesh filename=package://biped_bike_runtime/meshes/l_foot_roll.STL
- link l_hip_pitch: geometry collision mesh filename=package://biped_bike_runtime/meshes/l_hip_pitch.STL; visual mesh filename=package://biped_bike_runtime/meshes/l_hip_pitch.STL
- link l_hip_roll: geometry collision mesh filename=package://biped_bike_runtime/meshes/l_hip_roll.STL; visual mesh filename=package://biped_bike_runtime/meshes/l_hip_roll.STL
- link l_hip_yaw: geometry collision mesh filename=package://biped_bike_runtime/meshes/l_hip_yaw.STL; visual mesh filename=package://biped_bike_runtime/meshes/l_hip_yaw.STL
- link l_knee_pitch: geometry collision mesh filename=package://biped_bike_runtime/meshes/l_knee_pitch.STL; visual mesh filename=package://biped_bike_runtime/meshes/l_knee_pitch.STL
- link l_knee_pitch_wheel: geometry collision mesh filename=package://biped_bike_runtime/meshes/l_knee_pitch_wheel.STL; visual mesh filename=package://biped_bike_runtime/meshes/l_knee_pitch_wheel.STL
- link r_ankle_pitch: geometry collision mesh filename=package://biped_bike_runtime/meshes/r_ankle_pitch.STL; visual mesh filename=package://biped_bike_runtime/meshes/r_ankle_pitch.STL
- link r_foot_roll: geometry collision mesh filename=package://biped_bike_runtime/meshes/r_foot_roll.STL; visual mesh filename=package://biped_bike_runtime/meshes/r_foot_roll.STL
- link r_hip_pitch: geometry collision mesh filename=package://biped_bike_runtime/meshes/r_hip_pitch.STL; visual mesh filename=package://biped_bike_runtime/meshes/r_hip_pitch.STL
- link r_hip_roll: geometry collision mesh filename=package://biped_bike_runtime/meshes/r_hip_roll.STL; visual mesh filename=package://biped_bike_runtime/meshes/r_hip_roll.STL
- link r_hip_yaw: geometry collision mesh filename=package://biped_bike_runtime/meshes/r_hip_yaw.STL; visual mesh filename=package://biped_bike_runtime/meshes/r_hip_yaw.STL
- link r_knee_pitch: geometry collision mesh filename=package://biped_bike_runtime/meshes/r_knee_pitch.STL; visual mesh filename=package://biped_bike_runtime/meshes/r_knee_pitch.STL
- link r_knee_pitch_wheel: geometry collision mesh filename=package://biped_bike_runtime/meshes/r_knee_pitch_wheel.STL; visual mesh filename=package://biped_bike_runtime/meshes/r_knee_pitch_wheel.STL
Joints:
- joint arm_elbow_pitch_jnt: origin xyz=-0.092132 -0.077697 0.0002 rpy=0 0 0.34907 -> xyz=0.0415 -0.11315 0.0002 rpy=0 0 1.5708
- joint arm_shoulder_pitch_jnt: limit lower=-0.436332 upper=3.14159 effort=4.1 velocity=6.38 -> lower=-2.0944 upper=3.14159 effort=4.1 velocity=6.38
- joint arm_wrist_roll_jnt: axis 0.34202 0 -0.93969 -> 1 0 0; origin xyz=0.0432 -0.015 -0.0147 rpy=-1.5708 0 -1.9199 -> xyz=0.0432 -0.015 -0.0147 rpy=-1.5708 0 3.1416
- joint l_knee_pitch_wheel_jnt: limit effort=1.5 velocity=20.0 -> effort=1.5 velocity=6.38
- joint r_knee_pitch_wheel_jnt: limit effort=1.5 velocity=20.0 -> effort=1.5 velocity=6.38

Commit message: Improve physical hardware runtime and bike visualization

File: urdf/biped_bike_runtime.urdf (robot description, URDF)
Before this commit: robot biped_bike_runtime_print_ver6, 21 links, 20 joints
Joints:
- joint lidar_joint: origin xyz=-0.20 0 0.20 rpy=0 -1.3374 0 -> xyz=-0.225441 -0.070000 0.092983 rpy=0 -1.3374 0
